Commit message: Update g1_21 config

File: resources/robots/g1_description/g1_21dof_rev_1_0.urdf (robot description, URDF)
Before this commit: robot g1_21dof_rev_1_0, 39 links, 38 joints
Joints:
- joint left_elbow_joint: limit lower=-1.0472 upper=2.0944 effort=25 velocity=37 -> lower=-1.0472 upper=1.5 effort=25 velocity=37
- joint left_shoulder_pitch_joint: limit lower=-3.0892 upper=2.6704 effort=25 velocity=37 -> lower=-1.5 upper=1.5 effort=25 velocity=37
- joint left_shoulder_roll_joint: limit lower=-1.5882 upper=2.2515 effort=25 velocity=37 -> lower=-0.1 upper=2.2515 effort=25 velocity=37
- joint left_shoulder_yaw_joint: limit lower=-2.618 upper=2.618 effort=25 velocity=37 -> lower=-0.2 upper=1.6 effort=25 velocity=37
- joint right_elbow_joint: limit lower=-1.0472 upper=2.0944 effort=25 velocity=37 -> lower=-1.0472 upper=1.5 effort=25 velocity=37
- joint right_shoulder_pitch_joint: limit lower=-3.0892 upper=2.6704 effort=25 velocity=37 -> lower=-1.5 upper=1.5 effort=25 velocity=37
- joint right_shoulder_roll_joint: limit lower=-2.2515 upper=1.5882 effort=25 velocity=37 -> lower=-2.2515 upper=0.1 effort=25 velocity=37
- joint right_shoulder_yaw_joint: limit lower=-2.618 upper=2.618 effort=25 velocity=37 -> lower=-1.6 upper=0.2 effort=25 velocity=37
